Commit message: 7/31 update

File: isaacpjt/dongmin/M0609/doosan-robot2/urdf/m0609_isaac_sim.urdf (robot description, URDF)
Before this commit: robot m0609, 9 links, 8 joints
Links:
- link base_link: geometry collision mesh filename=meshes/m0609_collision/MF0609_0_0.dae scale=0.001 0.001 0.001; visual mesh filename=meshes/m0609_white/MF0609_0_0.dae scale=0.001 0.001 0.001
- link link_1: geometry collision mesh filename=meshes/m0609_collision/MF0609_1_0.dae scale=0.001 0.001 0.001; visual mesh filename=meshes/m0609_white/MF0609_1_0.dae scale=0.001 0.001 0.001
- link link_2: geometry collision mesh filename=meshes/m0609_collision/MF0609_2_0.dae scale=0.001 0.001 0.001; collision mesh filename=meshes/m0609_collision/MF0609_2_1.dae scale=0.001 0.001 0.001
- link link_3: geometry collision mesh filename=meshes/m0609_collision/MF0609_3_0.dae scale=0.001 0.001 0.001; visual mesh filename=meshes/m0609_white/MF0609_3_0.dae scale=0.001 0.001 0.001
- link link_4: geometry collision mesh filename=meshes/m0609_collision/MF0609_4_0.dae scale=0.001 0.001 0.001; collision mesh filename=meshes/m0609_collision/MF0609_4_1.dae scale=0.001 0.001 0.001
- link link_5: geometry collision mesh filename=meshes/m0609_collision/MF0609_5_0.dae scale=0.001 0.001 0.001; visual mesh filename=meshes/m0609_white/MF0609_5_0.dae scale=0.001 0.001 0.001
- link link_6: geometry collision mesh filename=meshes/m0609_collision/MF0609_6_0.dae scale=0.001 0.001 0.001; visual mesh filename=meshes/m0609_white/MF0609_6_0.dae scale=0.001 0.001 0.001
